File: pcb/pcb/krunchpad-20.kicad_pcb (KiCad board)
At the start: 2 copper layers, 100 x 97.9 mm, 49 parts, among them J1 Conn_01x04_Socket, SW1 SW_Push_45deg, SW10 SW_Push_45deg, SW11 SW_Push_45deg, SW12 SW_Push_45deg, SW13 SW_Push_45deg, SW14 SW_Push_45deg, SW15 SW_Push_45deg, SW16 SW_Push_45deg, SW17 SW_Push_45deg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

Commit message: Changed oled socket to SMD, added extra slot for 128x64 oled, updated relevent info info in BOM, updated images
Parts:
- removed the REF** at (121.9, 11.3)
- removed the REF** at (30.3, 11.1)
- added J2: Conn_01x04_Socket, Connector_PinSocket_2.54mm:PinSocket_1x04_P2.54mm_Vertical_SMD_Pin1Left, F.Cu at (51.5, 27.0)
- added REF**: MountingHole_2.2mm_M2_Pad_TopBottom, MountingHole:MountingHole_2.2mm_M2_Pad_TopBottom, F.Cu at (121.9, 11.3)
- added REF**: MountingHole_2.2mm_M2_Pad_TopBottom, MountingHole:MountingHole_2.2mm_M2_Pad_TopBottom, F.Cu at (30.3, 11.1)
- J1: footprint 0.91-OLED:SSD1306-0.91-OLED-4pin-128x32 -> Connector_PinSocket_2.54mm:PinSocket_1x04_P2.54mm_Vertical_SMD_Pin1Left
- moved J1 36.7 mm to (35.0, 17.5)
Routing:
- net SDA: track 45.3 -> 68.2 mm
- net SCL: track 45.3 -> 60.8 mm
- net +3V3: track 68.1 -> 71.9 mm
- net C2: track 127.6 -> 130.8 mm, vias 1 -> 0
- net R1: track 100.7 -> 102.4 mm
- net GND: track 70.5 -> 69.9 mm
Other:
- board text added: "krunchpad v2"

Commit message: updated pcb file with rotary encoder, updated gerber and case
Parts:
- added G***: LOGO, LOGO, B.Cu at (53.4, 17.3)
- added JP1: SolderJumper_2_Bridged, Jumper:SolderJumper-2_P1.3mm_Bridged_RoundedPad1.0x1.5mm, B.Cu at (81.3, 20.1)
- added JP2: SolderJumper_2_Bridged, Jumper:SolderJumper-2_P1.3mm_Bridged_RoundedPad1.0x1.5mm, B.Cu at (81.3, 22.7)
- added SW21: RotaryEncoder_Switch, Rotary_Encoder:RotaryEncoder_Alps_EC11E-Switch_Vertical_H20mm, F.Cu at (101.4, 15.2)
- moved G*** 55.5 mm to (47.9, 17.4)
- moved logo1 55.5 mm to (61.6, 17.4)
Connections:
- net SCL renamed GP7/SCL
- net SDA renamed GP6/SDA
Routing:
- net Net-(JP1-B): track 0.00 -> 23.0 mm, vias 0 -> 1
- net Net-(JP2-A): track 0.00 -> 20.5 mm, vias 0 -> 1
- net GND: track 69.9 -> 80.1 mm
- net GP6/SDA: track 68.2 -> 70.8 mm
- net GP7/SCL: track 60.8 -> 63.3 mm
